Commit message: 新ブランチ作成時のコンフリクト解消

File: robots/hydrus_xi/urdf/common.xacro (robot description, xacro)
@@ -39,4 +39,90 @@
     </collision>
   </xacro:macro>
+#<<<<<<< Updated upstream
+#=======
+  <!--   <joint name="joint_eff" type="fixed"> -->
+  <!--     <parent link="link4"/> -->
+  <!--     <child link="end_effector"/> -->
+  <!--     <origin rpy="0 0 0" xyz="${link_length} 0 0.04"/> -->
+  <!-- </joint> -->
+  <!-- <link name="end_effector">
+    <inertial>
+      <origin xyz="0 0 0" rpy="0 0 0"/>
+      <mass value="0.001"/>
+      <inertia
+          ixx="0.0001" ixy="0.0" ixz="0.0"
+          iyy="0.0001" iyz="0.0"
+          izz="0.0001"/>
+    </inertial>
+      <collision>
+        <origin rpy="0 0 0" xyz="0 0 0"/>
+        <geometry>
+          <sphere radius="0.02"/>
+        </geometry>
+      </collision>
+      <visual>
+        <origin rpy="0 0 0" xyz="0 0 0"/>
+        <geometry>
+          <sphere radius="0.02"/>
+        </geometry>
+      </visual>
+  </link>  -->
+  <!-- <link name="end_effector"> -->
+  <!--   <inertial> -->
+  <!--     <origin xyz="0.00 0 0" rpy="0 0 1.57"/> -->
+  <!--     <mass value="0.02"/> -->
+  <!--     <inertia -->
+  <!--         ixx="1e-6" ixy="0.0" ixz="0.0" -->
+  <!--         iyy="1e-6" iyz="0.0" -->
+  <!--         izz="1e-6"/> -->
+  <!--   </inertial> -->
+  <!--     <collision> -->
+  <!--       <origin rpy="0 1.57 0" xyz="0.1 0 0"/> -->
+  <!--       <geometry> -->
+  <!--         <cylinder length="0.2" radius="0.01"/> -->
+  <!--       </geometry> -->
+  <!--     </collision> -->
+  <!--     <visual> -->
+  <!--       <origin rpy="0 1.57 0" xyz="0.1 0 0"/> -->
+  <!--       <geometry> -->
+  <!--         <cylinder length="0.2" radius="0.01"/> -->
+  <!--       </geometry> -->
+  <!--     </visual> -->
+  <!--     <visual> -->
+  <!--       <origin rpy="0 0 0" xyz="0.2 0 0"/> -->
+  <!--       <geometry> -->
+  <!--         <sphere radius="0.01"/> -->
+  <!--       </geometry> -->
+  <!--     </visual> -->
+  <!-- </link> -->
+  <!-- <joint name="end_eff" type="fixed"> -->
+  <!--     <parent link="end_effector"/> -->
+  <!--     <child link="end_frame"/> -->
+  <!--     <origin rpy="0 0 0" xyz="0.2 0 0"/> -->
+  <!-- </joint> -->
+  <!-- <link name="end_frame"> -->
+  <!--     <collision> -->
+  <!--       <origin rpy="0 0 0" xyz="0 0 0"/> -->
+  <!--       <geometry> -->
+  <!--         <sphere radius="0.01"/> -->
+  <!--       </geometry> -->
+  <!--     </collision> -->
+  <!-- </link> -->
+  <!-- <gazebo reference="end_frame"> -->
+  <!--   <sensor name="contacts" type="contact"> -->
+  <!--       <contact> -->
+  <!--         <collision>link4_fixed_joint_lump__end_frame_collision_2</collision> -->
+  <!--       </contact> -->
+  <!--       <plugin name="gazebo_ros_bumper_controller" filename="libgazebo_ros_bumper.so"> -->
+  <!--         <always_on>true</always_on> -->
+  <!--         <robotNamespace>/hydrus_xi</robotNamespace> -->
+  <!--         <bumperTopicName>bumper_states</bumperTopicName> -->
+  <!--         <frameName>bumper</frameName> -->
+  <!--         <visualize>true</visualize> -->
+  <!--         <update_rate>1000.0</update_rate>         -->
+  <!--       </plugin> -->
+  <!--   </sensor> -->
+  <!-- </gazebo> -->
+#>>>>>>> Stashed changes
   <xacro:macro name="extra_module" params="name parent *origin *inertial visible:=0 model_url:=0">
     <joint name="${parent}2${name}" type="fixed">

Commit message: 直近の変更と同じ

File: robots/hydrus_xi/urdf/common.xacro (robot description, xacro)
@@ -39,95 +39,4 @@
     </collision>
   </xacro:macro>
-#<<<<<<< Updated upstream
-#<<<<<<< Updated upstream
-#=======
-#=======
-#>>>>>>> Stashed changes
-  <!--   <joint name="joint_eff" type="fixed"> -->
-  <!--     <parent link="link4"/> -->
-  <!--     <child link="end_effector"/> -->
-  <!--     <origin rpy="0 0 0" xyz="${link_length} 0 0.04"/> -->
-  <!-- </joint> -->
-  <!-- <link name="end_effector">
-    <inertial>
-      <origin xyz="0 0 0" rpy="0 0 0"/>
-      <mass value="0.001"/>
-      <inertia
-          ixx="0.0001" ixy="0.0" ixz="0.0"
-          iyy="0.0001" iyz="0.0"
-          izz="0.0001"/>
-    </inertial>
-      <collision>
-        <origin rpy="0 0 0" xyz="0 0 0"/>
-        <geometry>
-          <sphere radius="0.02"/>
-        </geometry>
-      </collision>
-      <visual>
-        <origin rpy="0 0 0" xyz="0 0 0"/>
-        <geometry>
-          <sphere radius="0.02"/>
-        </geometry>
-      </visual>
-  </link>  -->
-  <!-- <link name="end_effector"> -->
-  <!--   <inertial> -->
-  <!--     <origin xyz="0.00 0 0" rpy="0 0 1.57"/> -->
-  <!--     <mass value="0.02"/> -->
-  <!--     <inertia -->
-  <!--         ixx="1e-6" ixy="0.0" ixz="0.0" -->
-  <!--         iyy="1e-6" iyz="0.0" -->
-  <!--         izz="1e-6"/> -->
-  <!--   </inertial> -->
-  <!--     <collision> -->
-  <!--       <origin rpy="0 1.57 0" xyz="0.1 0 0"/> -->
-  <!--       <geometry> -->
-  <!--         <cylinder length="0.2" radius="0.01"/> -->
-  <!--       </geometry> -->
-  <!--     </collision> -->
-  <!--     <visual> -->
-  <!--       <origin rpy="0 1.57 0" xyz="0.1 0 0"/> -->
-  <!--       <geometry> -->
-  <!--         <cylinder length="0.2" radius="0.01"/> -->
-  <!--       </geometry> -->
-  <!--     </visual> -->
-  <!--     <visual> -->
-  <!--       <origin rpy="0 0 0" xyz="0.2 0 0"/> -->
-  <!--       <geometry> -->
-  <!--         <sphere radius="0.01"/> -->
-  <!--       </geometry> -->
-  <!--     </visual> -->
-  <!-- </link> -->
-  <!-- <joint name="end_eff" type="fixed"> -->
-  <!--     <parent link="end_effector"/> -->
-  <!--     <child link="end_frame"/> -->
-  <!--     <origin rpy="0 0 0" xyz="0.2 0 0"/> -->
-  <!-- </joint> -->
-  <!-- <link name="end_frame"> -->
-  <!--     <collision> -->
-  <!--       <origin rpy="0 0 0" xyz="0 0 0"/> -->
-  <!--       <geometry> -->
-  <!--         <sphere radius="0.01"/> -->
-  <!--       </geometry> -->
-  <!--     </collision> -->
-  <!-- </link> -->
-  <!-- <gazebo reference="end_frame"> -->
-  <!--   <sensor name="contacts" type="contact"> -->
-  <!--       <contact> -->
-  <!--         <collision>link4_fixed_joint_lump__end_frame_collision_2</collision> -->
-  <!--       </contact> -->
-  <!--       <plugin name="gazebo_ros_bumper_controller" filename="libgazebo_ros_bumper.so"> -->
-  <!--         <always_on>true</always_on> -->
-  <!--         <robotNamespace>/hydrus_xi</robotNamespace> -->
-  <!--         <bumperTopicName>bumper_states</bumperTopicName> -->
-  <!--         <frameName>bumper</frameName> -->
-  <!--         <visualize>true</visualize> -->
-  <!--         <update_rate>1000.0</update_rate>         -->
-  <!--       </plugin> -->
-  <!--   </sensor> -->
-  <!-- </gazebo> -->
-#<<<<<<< Updated upstream
-#>>>>>>> Stashed changes
-#>>>>>>> Stashed changes
   <xacro:macro name="extra_module" params="name parent *origin *inertial visible:=0 model_url:=0">
     <joint name="${parent}2${name}" type="fixed">
