Commit message: dynamics damping="0.05 55

File: robots/hydrus_xi/urdf/branch_type_link.urdf.xacro (robot description, xacro)
@@ -48,5 +48,5 @@
       <origin rpy="0 0 0" xyz="0.1555 0.0 0.015"/>
       <axis xyz="0 0 1"/>
-      <dynamics damping="0.8" friction="0.0"/>
+      <dynamics damping="0.05" friction="0.0"/>
     </joint>
     <joint name="joint${child2}" type="revolute">

Commit message: <dynamics damping="0.05" friction="0.0"/>

File: robots/hydrus_xi/urdf/branch_type_link.urdf.xacro (robot description, xacro)
@@ -64,5 +64,5 @@
       <origin rpy="0 0 ${pi * 4.0 / 3.0}" xyz="-0.07775 -0.13467 0.015"/>
       <axis xyz="0 0 1"/>
-      <dynamics damping="0.8" friction="0.0"/>
+      <dynamics damping="0.05" friction="0.0"/>
     </joint>
     #### hardware interface ####

Commit message: urdf表記統一

File: robots/hydrus_xi/urdf/branch_type_link.urdf.xacro (robot description, xacro)
@@ -194,5 +194,5 @@
         <origin rpy="0 0 0" xyz="${link_length} 0 0"/>
         <axis xyz="0 0 1"/>
-        <dynamics damping="0.8" friction="0.0"/>
+        <dynamics damping="0.05" friction="0.0"/>
       </joint>
     </xacro:unless>

Commit message: joint2のURDFもいじった

File: robots/hydrus_xi/urdf/branch_type_link.urdf.xacro (robot description, xacro)
@@ -56,5 +56,5 @@
       <origin rpy="0 0 ${pi * 2.0 / 3.0}" xyz="-0.07775 0.13467 0.015"/>
       <axis xyz="0 0 1"/>
-      <dynamics damping="0.8" friction="0.0"/>
+      <dynamics damping="0.05" friction="0.0"/>
     </joint>
     <joint name="joint${child3}" type="revolute">

Commit message: 0.8にした

File: robots/hydrus_xi/urdf/branch_type_link.urdf.xacro (robot description, xacro)
@@ -56,5 +56,5 @@
       <origin rpy="0 0 ${pi * 2.0 / 3.0}" xyz="-0.07775 0.13467 0.015"/>
       <axis xyz="0 0 1"/>
-      <dynamics damping="0.05" friction="0.0"/>
+      <dynamics damping="0.8" friction="0.0"/>
     </joint>
     <joint name="joint${child3}" type="revolute">

Commit message: damping 0.2

File: robots/hydrus_xi/urdf/branch_type_link.urdf.xacro (robot description, xacro)
@@ -48,5 +48,5 @@
       <origin rpy="0 0 0" xyz="0.1555 0.0 0.015"/>
       <axis xyz="0 0 1"/>
-      <dynamics damping="0.05" friction="0.0"/>
+      <dynamics damping="0.20" friction="0.0"/>
     </joint>
     <joint name="joint${child2}" type="revolute">
@@ -64,5 +64,5 @@
       <origin rpy="0 0 ${pi * 4.0 / 3.0}" xyz="-0.07775 -0.13467 0.015"/>
       <axis xyz="0 0 1"/>
-      <dynamics damping="0.05" friction="0.0"/>
+      <dynamics damping="0.20" friction="0.0"/>
     </joint>
     #### hardware interface ####

File: robots/hydrus_xi/urdf/link.urdf.xacro (robot description, xacro)
@@ -129,5 +129,5 @@
         <origin rpy="0 0 0" xyz="${link_length} 0 0"/>
         <axis xyz="0 0 1"/>
-        <dynamics damping="0.05" friction="0.05"/>
+        <dynamics damping="0.20" friction="0.05"/>
       </joint>
     </xacro:unless>

Commit message: Y時の方のURDFをもとに戻した

File: robots/hydrus_xi/urdf/branch_type_link.urdf.xacro (robot description, xacro)
@@ -48,5 +48,5 @@
       <origin rpy="0 0 0" xyz="0.1555 0.0 0.015"/>
       <axis xyz="0 0 1"/>
-      <dynamics damping="0.20" friction="0.0"/>
+      <dynamics damping="0.80" friction="0.0"/>
     </joint>
     <joint name="joint${child2}" type="revolute">
@@ -64,5 +64,5 @@
       <origin rpy="0 0 ${pi * 4.0 / 3.0}" xyz="-0.07775 -0.13467 0.015"/>
       <axis xyz="0 0 1"/>
-      <dynamics damping="0.20" friction="0.0"/>
+      <dynamics damping="0.80" friction="0.0"/>
     </joint>
     #### hardware interface ####

File: robots/hydrus_xi/urdf/link.urdf.xacro (robot description, xacro)
@@ -129,5 +129,5 @@
         <origin rpy="0 0 0" xyz="${link_length} 0 0"/>
         <axis xyz="0 0 1"/>
-        <dynamics damping="0.20" friction="0.05"/>
+        <dynamics damping="0.10" friction="0.05"/>
       </joint>
     </xacro:unless>
