Commit message: dynamics damping="0.05" friction="0.05" 140(0.8)

File: robots/hydrus_xi/urdf/link.urdf.xacro (robot description, xacro)
@@ -129,5 +129,5 @@
         <origin rpy="0 0 0" xyz="${link_length} 0 0"/>
         <axis xyz="0 0 1"/>
-        <dynamics damping="0.8" friction="0.05"/>
+        <dynamics damping="0.05" friction="0.05"/>
       </joint>
     </xacro:unless>

Commit message: コメント追加

File: robots/hydrus_xi/urdf/link.urdf.xacro (robot description, xacro)
@@ -129,5 +129,5 @@
         <origin rpy="0 0 0" xyz="${link_length} 0 0"/>
         <axis xyz="0 0 1"/>
-        <dynamics damping="0.05" friction="0.05"/>
+        <dynamics damping="0.05" friction="0.05"/>//もとは0.8
       </joint>
     </xacro:unless>

Commit message: //もとは0.8 を削除

File: robots/hydrus_xi/urdf/link.urdf.xacro (robot description, xacro)
@@ -129,5 +129,5 @@
         <origin rpy="0 0 0" xyz="${link_length} 0 0"/>
         <axis xyz="0 0 1"/>
-        <dynamics damping="0.05" friction="0.05"/>//もとは0.8
+        <dynamics damping="0.05" friction="0.05"/>
       </joint>
     </xacro:unless>

Commit message: dynamics damping="0.05

File: robots/hydrus_xi/urdf/link.urdf.xacro (robot description, xacro)
@@ -129,5 +129,5 @@
         <origin rpy="0 0 0" xyz="${link_length} 0 0"/>
         <axis xyz="0 0 1"/>
-        <dynamics damping="0.10" friction="0.05"/>
+        <dynamics damping="0.05" friction="0.05"/>
       </joint>
     </xacro:unless>
