Commit message: dynamics damping="0.1"

File: robots/hydrus_xi/urdf/link.urdf.xacro (robot description, xacro)
@@ -129,5 +129,5 @@
         <origin rpy="0 0 0" xyz="${link_length} 0 0"/>
         <axis xyz="0 0 1"/>
-        <dynamics damping="0.05" friction="0.05"/>
+        <dynamics damping="0.1" friction="0.05"/>
       </joint>
     </xacro:unless>

Commit message: dynamics damping="0.05"

File: robots/hydrus_xi/urdf/link.urdf.xacro (robot description, xacro)
@@ -129,5 +129,5 @@
         <origin rpy="0 0 0" xyz="${link_length} 0 0"/>
         <axis xyz="0 0 1"/>
-        <dynamics damping="0.1" friction="0.05"/>
+        <dynamics damping="0.05" friction="0.05"/>
       </joint>
     </xacro:unless>

Commit message: friction="0.01"

File: robots/hydrus_xi/urdf/link.urdf.xacro (robot description, xacro)
@@ -129,5 +129,5 @@
         <origin rpy="0 0 0" xyz="${link_length} 0 0"/>
         <axis xyz="0 0 1"/>
-        <dynamics damping="0.05" friction="0.05"/>
+        <dynamics damping="0.05" friction="0.01"/>
       </joint>
     </xacro:unless>

Commit message: back urdf

File: robots/hydrus_xi/urdf/link.urdf.xacro (robot description, xacro)
@@ -129,5 +129,5 @@
         <origin rpy="0 0 0" xyz="${link_length} 0 0"/>
         <axis xyz="0 0 1"/>
-        <dynamics damping="0.05" friction="0.01"/>
+        <dynamics damping="0.05" friction="0.05"/>
       </joint>
     </xacro:unless>
